File: S0_SchematicData/SchematicLayout_Basic/SchematicLayout.kicad_sch (KiCad schematic)
At the start: 12 parts, among them P1 Conn_Plug_2P, U1 LMZM23600V5, U2 ESP32-S2-WROVER

Commit message: Model updates and schematic changes
Further progress on line creation and new grasshopper scripts to assist with modelling. Also using individual python files for the svg extraction. Misc. changes
Connections:
- net at Vancouver.4 (BA): no longer U2.14 (IO11)
- net at Vancouver.5 (GA): no longer U2.13 (IO10)
- net at Vancouver.6 (RA): no longer U2.12 (IO09)
- net at U2.10 (IO07): no longer Dundee.5 (GA)
- net at U2.11 (IO08): no longer Dundee.4 (BA)
- net at U2.3 (IO00): no longer Auerbach.6 (RA)
- net at U2.39 (IO45): no longer Dial_PowerIntensityLED.1
- net at U2.4 (IO01): no longer Auerbach.5 (GA)
- net at U2.40 (IO46): no longer Dial_PowerIntensityLED.3
- net at U2.5 (IO02): no longer Auerbach.4 (BA)
- net at U2.6 (IO03): no longer Salina.6 (RA)
- net at U2.7 (IO04): no longer Salina.4 (BA)
- net at U2.8 (IO05): no longer Salina.5 (GA)
- net at U2.9 (IO06): no longer Dundee.6 (RA)
Other:
- note removed: "TODO: Find away to control the power intensity of each LED individually using a potentiaometer that the ESP32 can drive through an anolog signal, or some sort of signal"
